File: PCB_Maker/PCB_Maker.kicad_sch (KiCad schematic)
At the start: 55 parts, among them J1 USB_C_Receptacle_USB2.0_16P, J10 Conn_02x07_Odd_Even, J11 Conn_01x02, J12 Conn_01x06, J2 Conn_ST_STDC14, J3 Conn_01x02, J4 Conn_01x04, J5 Conn_01x04, J6 Conn_01x05, J7 Conn_01x03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

Commit message: PCB improve
Connections:
- net 3.3V is gone; now on net +3.3V: R4.1
Changed lines of the file:
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@@
 		)
 	)
-	(label "3.3V"
+	(label "+3.3V"
 		(at 69.85 74.93 270)
 		(fields_autoplaced yes)
