File: PCB_Maker/_autosave-PCB_Maker.kicad_sch (KiCad schematic)
At the start: 56 parts, among them J1 USB_C_Receptacle_USB2.0_16P, J10 Conn_02x07_Odd_Even, J11 Conn_01x02, J12 Conn_01x06, J2 Conn_ST_STDC14, J3 Conn_01x02, J4 Conn_01x04, J5 Conn_01x04, J6 Conn_01x05, J7 Conn_01x03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

Commit message: pcb correction
Parts:
- removed C5: 1u, Capacitor_SMD:C_0402_1005Metric_Pad0.74x0.62mm_HandSolder, symbol Device:C_Small
- added C5: 47u, Capacitor_SMD:C_0402_1005Metric_Pad0.74x0.62mm_HandSolder, symbol Device:C
Connections:
- net +3.3V: now also C5.1; no longer C6.1
- net +5V: now also C6.1
- net GND: now also C5.2
Changed lines of the file:
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@@
 	)
 	(junction
+		(at 257.81 52.07)
+		(diameter 0)
+		(color 0 0 0 0)
+	)
+	(junction
 		(at 57.15 130.81)
 		(diameter 0)
@@
 	)
 	(junction
+		(at 267.97 29.21)
+		(diameter 0)
+		(color 0 0 0 0)
+	)
+	(junction
 		(at 246.38 52.07)
 		(diameter 0)
@@
 	(wire
 		(pts
-			(xy 264.16 29.21) (xy 257.81 29.21)
+			(xy 270.51 29.21) (xy 267.97 29.21)
 		)
 		(stroke
@@
 	(wire
 		(pts
+			(xy 267.97 52.07) (xy 257.81 52.07)
+		)
+		(stroke
+			(width 0)
+			(type default)
+		)
+	)
+	(wire
+		(pts
 			(xy 254 39.37) (xy 257.81 39.37)
 		)
@@
 	(wire
 		(pts
+			(xy 267.97 43.18) (xy 267.97 52.07)
+		)
+		(stroke
+			(width 0)
+			(type default)
+		)
+	)
+	(wire
+		(pts
 			(xy 173.99 24.13) (xy 173.99 29.21)
 		)
@@
 	(wire
 		(pts
+			(xy 267.97 29.21) (xy 257.81 29.21)
+		)
+		(stroke
+			(width 0)
+			(type default)
+		)
+	)
+	(wire
+		(pts
 			(xy 128.27 111.76) (xy 134.62 111.76)
 		)
@@
 		)
 	)
+	(wire
+		(pts
+			(xy 267.97 29.21) (xy 267.97 35.56)
+		)
+		(stroke
+			(width 0)
+			(type default)
+		)
+	)
 	(polyline
 		(pts
@@
 	(symbol
 		(lib_id "power:+3.3V")
-		(at 264.16 29.21 270)
+		(at 270.51 29.21 270)
 		(unit 1)
 		(exclude_from_sim no)
@@
 		(dnp no)
 		(property "Reference" "#PWR023"
-			(at 260.35 29.21 0)
+			(at 266.7 29.21 0)
 			(effects
 				(font
@@
 		)
 		(property "Value" "+3.3V"
-			(at 267.97 29.2099 90)
+			(at 274.32 29.2099 90)
 			(effects
 				(font
@@
 		)
 		(property "Footprint" ""
-			(at 264.16 29.21 0)
+			(at 270.51 29.21 0)
 			(effects
 				(font
@@
 		)
 		(property "Datasheet" ""
-			(at 264.16 29.21 0)
+			(at 270.51 29.21 0)
 			(effects
 				(font
@@
 		)
 		(property "Description" "Power symbol creates a global label with name \"+3.3V\""
-			(at 264.16 29.21 0)
+			(at 270.51 29.21 0)
 			(effects
 				(font
@@
 			)
 		)
-		(property "Value" "+3.3V"
+		(property "Value" "+5V"
 			(at 171.45 74.93 0)
 			(effects
@@
 	)
 	(symbol
+		(lib_id "Device:C")
+		(at 267.97 39.37 0)
+		(unit 1)
+		(exclude_from_sim no)
+		(in_bom yes)
+		(on_board yes)
+		(dnp no)
+		(property "Reference" "C5"
+			(at 264.668 39.37 90)
+			(effects
+				(font
+					(size 1.27 1.27)
+				)
+			)
+		)
+		(property "Value" "47u"
+			(at 271.272 39.116 90)
+			(effects
+				(font
+					(size 1.27 1.27)
+				)
+			)
+		)
+		(property "Footprint" "Capacitor_SMD:C_0402_1005Metric_Pad0.74x0.62mm_HandSolder"
+			(at 268.9352 43.18 0)
+			(effects
+				(font
+					(size 1.27 1.27)
+				)
+				(hide yes)
+			)
+		)
+		(property "Datasheet" "~"
+			(at 267.97 39.37 0)
+			(effects
+				(font
+					(size 1.27 1.27)
+				)
+				(hide yes)
+			)
+		)
+		(property "Description" "Unpolarized capacitor"
+			(at 267.97 39.37 0)
+			(effects
+				(font
+					(size 1.27 1.27)
+				)
+				(hide yes)
+			)
+		)
+		(pin "1"
+		)
+		(pin "2"
+		)
+		(instances
+			(project "PCB_Maker"
+				(path "/8c89adab-4772-459d-bb0d-6509137ae624"
+					(reference "C5")
+					(unit 1)
+				)
+			)
+		)
+	)
+	(symbol
 		(lib_id "power:GND")
 		(at 57.15 132.08 0)
@@
 					(unit 1)
 				)
-			)
-		)
-	)
-	(symbol
-		(lib_id "Device:C_Small")
-		(at 156.21 55.88 0)
-		(unit 1)
-		(exclude_from_sim no)
-		(in_bom yes)
-		(on_board yes)
-		(dnp no)
-		(fields_autoplaced yes)
-		(property "Reference" "C5"
-			(at 158.75 54.6163 0)
-			(effects
-				(font
-					(size 1.27 1.27)
-				)
-				(justify left)
-			)
-		)
-		(property "Value" "1u"
-			(at 158.75 57.1563 0)
-			(effects
-				(font
-					(size 1.27 1.27)
-				)
-				(justify left)
-			)
-		)
-		(property "Footprint" "Capacitor_SMD:C_0402_1005Metric_Pad0.74x0.62mm_HandSolder"
-			(at 156.21 55.88 0)
-			(effects
-				(font
-					(size 1.27 1.27)
-				)
-				(hide yes)
-			)
-		)
-		(property "Datasheet" "~"
-			(at 156.21 55.88 0)
-			(effects
-				(font
-					(size 1.27 1.27)
-				)
-				(hide yes)
-			)
-		)
-		(property "Description" ""
-			(at 156.21 55.88 0)
-			(effects
-				(font
-					(size 1.27 1.27)
-				)
-				(hide yes)
-			)
-		)
-		(pin "1"
-		)
-		(pin "2"
-		)
-		(instances
-			(project "PCB_Maker"
-				(path "/8c89adab-4772-459d-bb0d-6509137ae624"
-					(reference "C5")
-					(unit 1)
-				)
