File: PCB_Maker/PCB_Maker.kicad_pcb (KiCad board)
At the start: 4 copper layers, 81.5 x 29.8 mm, 56 parts, among them J1 USB_C_Receptacle_USB2.0_16P, J10 Conn_02x07_Odd_Even, J12 Conn_01x06, J3 Conn_01x02, SW1 SW_Push, U1 STM32G431CBTx, U3 171013801

Commit message: pcb correction
Parts:
- added C3: 10n, Capacitor_SMD:C_0603_1608Metric_Pad1.08x0.95mm_HandSolder, B.Cu at (70.2, 117.2)
- added C4: 1u, Capacitor_SMD:C_0603_1608Metric_Pad1.08x0.95mm_HandSolder, B.Cu at (72.5, 116.8)
- added C5: 47u, Capacitor_SMD:C_0402_1005Metric_Pad0.74x0.62mm_HandSolder, B.Cu at (98.2, 124.2)
- added C6: 1u, Capacitor_SMD:C_0402_1005Metric_Pad0.74x0.62mm_HandSolder, B.Cu at (90.2, 105.0)
- added L1: 39n, LED_SMD:LED_0805_2012Metric_Pad1.15x1.40mm_HandSolder, F.Cu at (69.5, 116.5)
- C12, C15, C16, C19: moved to B.Cu
- Maker Ares_Express: renamed from MAKER Ares_Express
- moved C12 30.1 mm to (92.5, 124.0), turned to 180 degrees
- moved C16 26.0 mm to (96.2, 124.5), turned to -90 degrees
- moved C15 21.7 mm to (100.3, 124.5), turned to -90 degrees
- moved C19 17.7 mm to (77.0, 124.8), turned to 180 degrees
- renumbered VCC to J11, Ultrasound to J5, Accelerometer to J6, D1 to Zener1, D2 to Zener2
Connections:
- C15 pad 1: VCC -> +3.3V
- C16 pad 1: VCC -> +3.3V
- U1 pad 21: +3.3V -> +3.3VA
Routing:
- net GND: track 51.5 -> 43.8 mm, vias 192 -> 190
- net +3.3VA: track 0.00 -> 6.89 mm, vias 0 -> 1
- net VCC: track 27.3 -> 24.5 mm, vias 4 -> 6
- net +5V: track 5.56 -> 7.56 mm
- net /PA_7: track 25.3 -> 23.6 mm
- net /PA_6: track 27.0 -> 25.3 mm
- net +3.3V: track 37.7 -> 39.0 mm, vias 10 -> 12
- net /PA_5: track 28.8 -> 27.6 mm
- net /PB2_LED_3: track 11.2 -> 12.3 mm
- net /PC_14: track 33.7 -> 32.7 mm
- net /PB1_LED_2: track 10.7 -> 11.5 mm
- net /PC_15: track 32.8 -> 32.1 mm

Commit message: PCB correction Mr.Papazoglou
Parts:
- removed C14, C17, C18: 10uF, Capacitor_SMD:CP_Elec_4x5.7
- removed R16: 110m, Resistor_SMD:R_0603_1608Metric_Pad0.98x0.95mm_HandSolder
- C10, C9: footprint Capacitor_SMD:C_0402_1005Metric_Pad0.74x0.62mm_HandSolder -> Capacitor_SMD:C_0603_1608Metric_Pad1.08x0.95mm_HandSolder
- C15, C16: value 100nF -> 100n
- C3: footprint Capacitor_SMD:C_0603_1608Metric_Pad1.08x0.95mm_HandSolder -> Capacitor_SMD:C_0402_1005Metric_Pad0.74x0.62mm_HandSolder
- C5: value 47u -> 1u
- H2: renamed from Maker Ares_Express
- J9: renamed from Buck 5V
- moved C5 23.4 mm to (111.5, 105.0), turned to 180 degrees
- moved U2 9.31 mm to (62.2, 119.3), turned to 90 degrees
- moved C3 0.89 mm to (69.7, 116.5), turned to 180 degrees
- moved R1 0.67 mm to (59.4, 120.8)
- moved R2 0.48 mm to (65.0, 120.9)
- renumbered Zener1 to D1, Zener2 to D2, ST-link to J2, Ecran to J4, Servo1 to J7, Servo2 to J8, USB to U2
Connections:
- C5 pad 1: +3.3V -> +5V
- R14 pad 1: +5V -> +3.3V
- U2 pad 1: /D+ -> /D-
- U2 pad 3: /USB_DP -> /D+
- U2 pad 4: /USB_DM -> /USB_DP
- U2 pad 6: /D- -> /USB_DM
Routing:
- net VCC: track 24.5 -> 9.43 mm
- net /D+: track 16.6 -> 3.78 mm
- net /USB_DM: track 11.1 -> 22.1 mm, vias 2 -> 0
- net /USB_DP: track 10.5 -> 20.6 mm
- net /D-: track 14.3 -> 4.51 mm, vias 2 -> 0
- net GND: track 43.8 -> 35.7 mm, vias 190 -> 183
- net /I2C1_SCL: track 23.0 -> 17.3 mm
- net /PA_5: track 27.6 -> 22.1 mm
- net /I2C1_SDA: track 23.4 -> 18.4 mm
- net /PA_6: track 25.3 -> 21.0 mm
- net Net-(C14-Pad2): track 3.40 -> 0.00 mm
- net +5V: track 7.56 -> 10.8 mm, vias 4 -> 3
- net /PA_7: track 23.6 -> 20.6 mm
- net +3.3V: track 39.0 -> 41.9 mm, vias 12 -> 10
- net /PC_15: track 32.1 -> 33.5 mm, vias 2 -> 1
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