File: PCB_Maker_ancien/PCB_Maker.kicad_sch (KiCad schematic)
At the start: 56 parts, among them J1 USB_C_Receptacle_USB2.0_16P, J10 Conn_02x07_Odd_Even, J11 Conn_01x02, J12 Conn_01x06, J2 Conn_ST_STDC14, J3 Conn_01x02, J4 Conn_01x04, J5 Conn_01x04, J6 Conn_01x05, J7 Conn_01x03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

Commit message: PCB correction Mr.Papazoglou
Parts:
- C10, C9: footprint Capacitor_SMD:C_0603_1608Metric_Pad1.08x0.95mm_HandSolder -> Capacitor_SMD:C_0402_1005Metric_Pad0.74x0.62mm_HandSolder
- C15, C16: value 100n -> 100nF
- C3: footprint Capacitor_SMD:C_0402_1005Metric_Pad0.74x0.62mm_HandSolder -> Capacitor_SMD:C_0603_1608Metric_Pad1.08x0.95mm_HandSolder
Connections:
- net +3.3V: now also C5.1, C6.1; no longer R14.1
- net +5V: now also R14.1; no longer C5.1, C6.1
- net D+: now also U2.1 (I/O1); no longer U2.3 (I/O2)
- net D-: now also U2.6 (I/O1); no longer U2.1 (I/O1)
- net USB_DM: now also U2.4 (I/O2); no longer U2.6 (I/O1)
- net USB_DP: now also U2.3 (I/O2); no longer U2.4 (I/O2)
